Commit message: interfaces updated

File: interface_description/urdf/cat6.urdf.xacro (robot description, xacro)
@@ -3,22 +3,7 @@
        xmlns:ietf-network-topology="urn:ietf:params:xml:ns:yang:ietf-network-topology"
        xmlns:device-layer="urn:ietf:params:xml:ns:yang:device-layer"
-       xmlns:network-layer="urn:ietf:params:xml:ns:yang:network-layer"
+       xmlns:ethernet-port="urn:ietf:params:xml:ns:yang:ethernet-port"
        name="cat6">
-    <xacro:property name="cat6_yaml_file" value="$(find interface_description)/config/cat6.yaml" />
-    <xacro:property name="cat6_props" value="${xacro.load_yaml(cat6_yaml_file)}"/>
-    <xacro:property name="cat6_type" value="${cat6_props['wired-connection']['type']}"/>
-    <xacro:property name="cat6_length" value="${cat6_props['wired-connection']['length']}"/>
-    <xacro:property name="cat6_bandwidth" value="${cat6_props['wired-connection']['bandwidth']}"/>
-    <xacro:property name="cat6_jitter" value="${cat6_props['wired-connection']['jitter']}"/>
-    <xacro:property name="cat6_packet_loss" value="${cat6_props['wired-connection']['packet-loss']}"/>
-    <xacro:property name="cat6_reliability" value="${cat6_props['wired-connection']['reliability']}"/>
-    <xacro:property name="cat6_availability" value="${cat6_props['wired-connection']['availability']}"/>
-    <xacro:property name="cat6_qos_level" value="${cat6_props['wired-connection']['qos-level']}"/>
-    <xacro:property name="cat6_energy_efficiency" value="${cat6_props['wired-connection']['energy-efficiency']}"/>
-    <xacro:property name="cat6_compatibility" value="${cat6_props['wired-connection']['compatibility']}"/>
-    <xacro:property name="cat6_cost" value="${cat6_props['wired-connection']['cost']}"/>
-    <xacro:property name="cat6_scalability" value="${cat6_props['wired-connection']['scalability']}"/>
-    <xacro:property name="cat6_security_level" value="${cat6_props['wired-connection']['security-level']}"/>
-    <xacro:macro name="cat6" params="parent L2_network_id L1_network_id L2_id:=cat6_L2 L1_id:=cat6_L1">
+    <xacro:macro name="cat6" params="parent id:=0">
         <joint name="cat6_joint" type="fixed">
             <origin xyz="-1 1 0" rpy="0 0 0" />
@@ -43,31 +28,46 @@
             </collision>
         </link>
-    </xacro:macro>
-    <xacro:macro name="cat6_L2" params="id supporting_network supporting_node supporting_tp">
-        <ietf-network-topology:termination-point>
-            <tp-id>${id}</tp-id>
-            <supporting-termination-point>
-                <network-ref>${supporting_network}</network-ref>
-                <node-ref>${supporting_node}</node-ref>
-                <tp-ref>${supporting_tp}</tp-ref>
-            </supporting-termination-point>
-            <network-layer:network-layer-termination-point-attributes>
-                <tp-type>${cat6_type}</tp-type>
-                <bandwidth>${cat6_bandwidth}</bandwidth>
-                <jitter>${cat6_jitter}</jitter>
-                <packet_loss>${cat6_packet_loss}</packet_loss>
-                <reliability>${cat6_reliability}</reliability>
-                <cost>${cat6_cost}</cost>
-            </network-layer:network-layer-termination-point-attributes>
-        </ietf-network-topology:termination-point>
-    </xacro:macro>
-    <xacro:macro name="cat6_L1" params="id connector_type connector_format">
-        <ietf-network-topology:termination-point>
-            <tp-id>${id}</tp-id>
-            <device-layer:device-layer-termination-point-attributes>
-                <connector-type>${connector_type}</connector-type>
-                <connector-format>${connector_format}</connector-format>
-            </device-layer:device-layer-termination-point-attributes>
-        </ietf-network-topology:termination-point>
+        <yang>
+            <!-- cat6 network topology -->
+            <network>
+                <network-id>cat6-network</network-id>
+                <network-types>
+                    <dl:device-layer-topology xmlns:dl="urn:ietf:params:xml:ns:yang:device-layer"/>
+                </network-types>
+                <supporting-network>
+                    <network-ref>cat6-supporting-network</network-ref>
+                </supporting-network>
+                <node>
+                    <node-id>cat6-node</node-id>
+                    <supporting-node>
+                        <network-ref>cat6-supporting-network</network-ref>
+                        <node-ref>cat6-supporting-node</node-ref>
+                    </supporting-node>
+                    <dl:device-layer-node-attributes xmlns:dl="urn:ietf:params:xml:ns:yang:device-layer">
+                        <dl:device-name>cat6-interface</dl:device-name>
+                        <dl:device-type>port</dl:device-type>
+                    </dl:device-layer-node-attributes>
+                    <nt:termination-point xmlns:nt="urn:ietf:params:xml:ns:yang:ietf-network-topology">
+                        <nt:tp-id>tp-1</nt:tp-id>
+                        <nt:supporting-termination-point>
+                            <nt:network-ref>supporting-network-1</nt:network-ref>
+                            <nt:node-ref>supporting-node-1</nt:node-ref>
+                            <nt:tp-ref>tp-ref-1</nt:tp-ref>
+                        </nt:supporting-termination-point>
+                        <dl:device-layer-termination-point-attributes xmlns:dl="urn:ietf:params:xml:ns:yang:device-layer">
+                            <dl:port-name>port-1</dl:port-name>
+                            <dl:port-type>
+                                <eth:ethernet-port xmlns:eth="urn:ietf:params:xml:ns:yang:ethernet-port">
+                                <eth:port-id>eth1</eth:port-id>
+                                <eth:mac-address>00:1A:2B:3C:4D:5E</eth:mac-address>
+                                <eth:speed>1000Mbps</eth:speed>
+                                <eth:duplex-mode>full</eth:duplex-mode>
+                                </eth:ethernet-port>
+                            </dl:port-type>
+                        </dl:device-layer-termination-point-attributes>
+                    </nt:termination-point>
+                </node>
+            </network>
+        </yang>
     </xacro:macro>
 </robot>

File: interface_description/urdf/usb-typec.urdf.xacro (robot description, xacro)
@@ -4,16 +4,16 @@
        xmlns:device-layer="urn:ietf:params:xml:ns:yang:device-layer"
        xmlns:usb-port="urn:ietf:params:xml:ns:yang:usb-port"
-       name="usb30">
-    <xacro:macro name="usb30" params="parent id:=0">
-        <joint name="usb30_joint" type="fixed">
+       name="usb_typec">
+    <xacro:macro name="usb_typec" params="parent">
+        <joint name="usb_typec_joint" type="fixed">
             <origin xyz="-1 1 0" rpy="0 0 0" />
             <parent link="${parent}"/>
-            <child link="usb30_link"/>
+            <child link="usb-typec_link"/>
         </joint>
-        <link name="usb30_link">
+        <link name="usb_typec_link">
             <visual>
                 <origin rpy="0 0 0" xyz="0 0 0"/>
                 <geometry>
-                <mesh filename="package://interface_description/meshes/usb-A-female.stl" scale="0.001 0.001 0.001"/>
+                <mesh filename="package://interface_description/meshes/usb-typec-female.stl" scale="0.001 0.001 0.001"/>
                 </geometry>
                 <material name="LightGrey">
@@ -24,27 +24,27 @@
                 <origin xyz="0 0 0" rpy="0 0 0"/>
                 <geometry>
-                <mesh filename="package://interface_description/meshes/usb-A-female.stl" scale="0.001 0.001 0.001"/>
+                <mesh filename="package://interface_description/meshes/usb-typec-female.stl" scale="0.001 0.001 0.001"/>
                 </geometry>
             </collision>
         </link>
         <yang>
-            <!-- usb30 network topology -->
+            <!-- usb-typec network topology -->
             <network>
-                <network-id>usb30-network</network-id>
+                <network-id>usb-typec-network</network-id>
                 <network-types>
                     <dl:device-layer-topology xmlns:dl="urn:ietf:params:xml:ns:yang:device-layer"/>
                 </network-types>
                 <supporting-network>
-                    <network-ref>usb30-supporting-network</network-ref>
+                    <network-ref>usb-typec-supporting-network</network-ref>
                 </supporting-network>
                 <node>
-                    <node-id>usb30-node</node-id>
+                    <node-id>usb-typec-node</node-id>
                     <supporting-node>
-                        <network-ref>usb30-supporting-network</network-ref>
-                        <node-ref>usb30-supporting-node</node-ref>
+                        <network-ref>usb-typec-supporting-network</network-ref>
+                        <node-ref>usb-typec-supporting-node</node-ref>
                     </supporting-node>
                     <dl:device-layer-node-attributes xmlns:dl="urn:ietf:params:xml:ns:yang:device-layer">
-                        <dl:device-name>usb30-device</dl:device-name>
-                        <dl:device-type>usb30-port</dl:device-type>
+                        <dl:device-name>usb-typec-device</dl:device-name>
+                        <dl:device-type>usb-typec-port</dl:device-type>
                     </dl:device-layer-node-attributes>
                     <nt:termination-point xmlns:nt="urn:ietf:params:xml:ns:yang:ietf-network-topology">
@@ -59,6 +59,6 @@
                             <dl:port-type>
                                 <usb:usb-port xmlns:usb="urn:ietf:params:xml:ns:yang:usb-port">
-                                <usb:port-id>eth1</usb:port-id>
-                                <usb:version>USB3.0</usb:version>
+                                <usb:port-id>usb-typec</usb:port-id>
+                                <usb:version>USB3.2</usb:version>
                                 <usb:speed>5.00</usb:speed>
                                 <usb:power-consumption>2.5</usb:power-consumption>

Commit message: typoo fixed

File: interface_description/urdf/cat6.urdf.xacro (robot description, xacro)
@@ -15,5 +15,5 @@
                 <origin rpy="0 0 0" xyz="0 0 0"/>
                 <geometry>
-                <mesh filename="package://interface_description/meshes/rj45_female.stl" scale="0.001 0.001 0.001"/>
+                <mesh filename="package://interface_description/meshes/rj45-female.stl" scale="0.001 0.001 0.001"/>
                 </geometry>
                 <material name="LightGrey">
@@ -24,5 +24,5 @@
                 <origin xyz="0 0 0" rpy="0 0 0"/>
                 <geometry>
-                <mesh filename="package://interface_description/meshes/rj45_female.stl" scale="0.001 0.001 0.001"/>
+                <mesh filename="package://interface_description/meshes/rj45-female.stl" scale="0.001 0.001 0.001"/>
                 </geometry>
             </collision>

Commit message: yang content update

File: interface_description/urdf/cat6.urdf.xacro (robot description, xacro)
@@ -2,11 +2,11 @@
 <robot xmlns:xacro="http://ros.org/wiki/xacro"
        name="cat6">
-    <xacro:macro name="cat6" params="parent id:=0">
-        <joint name="cat6-${id}_joint" type="fixed">
-            <origin xyz="-1 1 0" rpy="0 0 0" />
+    <xacro:macro name="cat6" params="parent prefix id:=0 origin_xyz origin_rpy">
+        <joint name="${prefix}-cat6-${id}-joint" type="fixed">
+            <origin xyz="${origin_xyz}" rpy="${origin_rpy}" />
             <parent link="${parent}"/>
-            <child link="cat6-${id}_link"/>
+            <child link="${prefix}-cat6-${id}-link"/>
         </joint>
-        <link name="cat6-${id}_link">
+        <link name="${prefix}-cat6-${id}-link">
             <visual>
                 <origin rpy="0 0 0" xyz="0 0 0"/>
@@ -26,10 +26,10 @@
         </link>
         <nt:termination-point xmlns:nt="urn:ietf:params:xml:ns:yang:ietf-network-topology">
-            <nt:tp-id>tp-1</nt:tp-id>
+            <nt:tp-id>${prefix}-cat6-rj45-${id}</nt:tp-id>
             <dl:device-layer-termination-point-attributes xmlns:dl="urn:ietf:params:xml:ns:yang:device-layer">
                 <dl:port-name>rj45-${id}</dl:port-name>
                 <dl:port-type>rj45</dl:port-type>
                 <eth:ethernet-port xmlns:eth="urn:ietf:params:xml:ns:yang:ethernet-port">
-                    <eth:port-id>eth-${id}</eth:port-id>
+                    <eth:port-id>${prefix}-eth-${id}</eth:port-id>
                     <eth:mac-address>00:1A:2B:3C:4D:5E</eth:mac-address>
                     <eth:speed>1Gbps</eth:speed>

File: interface_description/urdf/usb-typec.urdf.xacro (robot description, xacro)
@@ -2,11 +2,11 @@
 <robot xmlns:xacro="http://ros.org/wiki/xacro"
        name="usb_typec">
-    <xacro:macro name="usb_typec" params="parent id=0">
-        <joint name="usb-typec-${id}_joint" type="fixed">
-            <origin xyz="-1 1 0" rpy="0 0 0" />
+    <xacro:macro name="usb_typec" params="parent prefix id:=0 origin_xyz origin_rpy">
+        <joint name="${prefix}-usb-typec-${id}-joint" type="fixed">
+            <origin xyz="${origin_xyz}" rpy="${origin_rpy}" />
             <parent link="${parent}"/>
-            <child link="usb-typec-${id}_link"/>
+            <child link="${prefix}-usb-typec-${id}-link"/>
         </joint>
-        <link name="usb-typec-${id}_link">
+        <link name="${prefix}-usb-typec-${id}-link">
             <visual>
                 <origin rpy="0 0 0" xyz="0 0 0"/>
@@ -26,10 +26,10 @@
         </link>
         <nt:termination-point xmlns:nt="urn:ietf:params:xml:ns:yang:ietf-network-topology">
-            <nt:tp-id>tp-1</nt:tp-id>
+            <nt:tp-id>${prefix}-usb-typec-${id}</nt:tp-id>
             <dl:device-layer-termination-point-attributes xmlns:dl="urn:ietf:params:xml:ns:yang:device-layer">
-                <dl:port-name>port-1</dl:port-name>
+                <dl:port-name>port-${id}</dl:port-name>
                 <dl:port-type>usb-c</dl:port-type>
                 <usb:usb-port xmlns:usb="urn:ietf:params:xml:ns:yang:usb-port">
-                    <usb:port-id>usb-typec-${id}</usb:port-id>
+                    <usb:port-id>${prefix}-usb-typec-${id}</usb:port-id>
                     <usb:version>USB3.2</usb:version>
                     <usb:speed>5.00</usb:speed>

File: interface_description/urdf/usb30.urdf.xacro (robot description, xacro)
@@ -2,11 +2,11 @@
 <robot xmlns:xacro="http://ros.org/wiki/xacro"
        name="usb30">
-    <xacro:macro name="usb30" params="parent id:=0">
-        <joint name="usb30-${id}_joint" type="fixed">
-            <origin xyz="-1 1 0" rpy="0 0 0" />
+    <xacro:macro name="usb30" params="parent prefix id:=0 origin_xyz origin_rpy">
+        <joint name="${prefix}-usb30-${id}-joint" type="fixed">
+            <origin xyz="${origin_xyz}" rpy="${origin_rpy}" />
             <parent link="${parent}"/>
-            <child link="usb30-${id}_link"/>
+            <child link="${prefix}-usb30-${id}-link"/>
         </joint>
-        <link name="usb30-${id}_link">
+        <link name="${prefix}-usb30-${id}-link">
             <visual>
                 <origin rpy="0 0 0" xyz="0 0 0"/>
@@ -26,11 +26,11 @@
         </link>
         <nt:termination-point xmlns:nt="urn:ietf:params:xml:ns:yang:ietf-network-topology">
-            <nt:tp-id>tp-1</nt:tp-id>
+            <nt:tp-id>${prefix}-usb30-${id}</nt:tp-id>
             <dl:device-layer-termination-point-attributes xmlns:dl="urn:ietf:params:xml:ns:yang:device-layer">
-                <dl:port-name>port-1</dl:port-name>
+                <dl:port-name>usb30-${id}</dl:port-name>
                 <dl:port-type>usb-a</dl:port-type>
                 <usb:usb-port xmlns:usb="urn:ietf:params:xml:ns:yang:usb-port">
-                    <usb:port-id>USB30-${id}</usb:port-id>
-                    <usb:version>USB3.0</usb:version>
+                    <usb:port-id>${prefix}-usb30-${id}</usb:port-id>
+                    <usb:version>usb3.0</usb:version>
                     <usb:speed>5.00</usb:speed>
                     <usb:power-consumption>2.5</usb:power-consumption>
