Commit message: params adjusted

File: interface_description/urdf/cat5e.urdf.xacro (robot description, xacro)
@@ -1,16 +1,16 @@
 <?xml version="1.0" encoding="UTF-8" ?>
 <robot xmlns:xacro="http://ros.org/wiki/xacro"
-       name="cat6">
-    <xacro:macro name="cat6" params="parent prefix id:=0 origin_xyz origin_rpy">
-        <joint name="${prefix}-cat6-${id}-joint" type="fixed">
+       name="cat5e">
+    <xacro:macro name="cat5e" params="parent prefix id:=0 origin_xyz origin_rpy">
+        <joint name="${prefix}-cat5e-${id}-joint" type="fixed">
             <origin xyz="${origin_xyz}" rpy="${origin_rpy}" />
             <parent link="${parent}"/>
-            <child link="${prefix}-cat6-${id}-link"/>
+            <child link="${prefix}-cat5e-${id}-link"/>
         </joint>
-        <link name="${prefix}-cat6-${id}-link">
+        <link name="${prefix}-cat5e-${id}-link">
             <visual>
                 <origin rpy="0 0 0" xyz="0 0 0"/>
                 <geometry>
-                <mesh filename="package://interface_description/meshes/rj45-female.stl" scale="0.001 0.001 0.001"/>
+                <mesh filename="package://interface_description/meshes/rj45_female.stl" scale="0.001 0.001 0.001"/>
                 </geometry>
                 <material name="LightGrey">
@@ -21,5 +21,5 @@
                 <origin xyz="0 0 0" rpy="0 0 0"/>
                 <geometry>
-                <mesh filename="package://interface_description/meshes/rj45-female.stl" scale="0.001 0.001 0.001"/>
+                <mesh filename="package://interface_description/meshes/rj45_female.stl" scale="0.001 0.001 0.001"/>
                 </geometry>
             </collision>

File: interface_description/urdf/usb-typec.urdf.xacro (robot description, xacro)
@@ -1,4 +1,5 @@
 <?xml version="1.0" encoding="UTF-8" ?>
 <robot xmlns:xacro="http://ros.org/wiki/xacro"
+       xmlns:usb="urn:ietf:params:xml:ns:yang:usb-port"
        name="usb_typec">
     <xacro:macro name="usb_typec" params="parent prefix id:=0 origin_xyz origin_rpy">
@@ -27,13 +28,12 @@
         <nt:termination-point xmlns:nt="urn:ietf:params:xml:ns:yang:ietf-network-topology">
             <nt:tp-id>${prefix}-usb-typec-${id}</nt:tp-id>
-            <dl:device-layer-termination-point-attributes xmlns:dl="urn:ietf:params:xml:ns:yang:device-layer">
-                <dl:port-name>port-${id}</dl:port-name>
-                <dl:port-type>usb-c</dl:port-type>
-                <usb:usb-port xmlns:usb="urn:ietf:params:xml:ns:yang:usb-port">
-                    <usb:port-id>${prefix}-usb-typec-${id}</usb:port-id>
-                    <usb:version>USB3.2</usb:version>
-                    <usb:speed>5.00</usb:speed>
-                    <usb:power-consumption>2.5</usb:power-consumption>
-                </usb:usb-port>
+            <dl:device-layer-termination-point-attributes
+                xmlns:dl="urn:ietf:params:xml:ns:yang:device-layer"
+                xmlns:usb="urn:ietf:params:xml:ns:yang:usb-port">
+                <dl:port-name>${prefix}-port</dl:port-name>
+                <dl:port-type>usb</dl:port-type>
+                <dl:wired>true</dl:wired>
+                <usb:version>usb3.2</usb:version>
+                <usb:power-consumption>2.5</usb:power-consumption>
             </dl:device-layer-termination-point-attributes>
         </nt:termination-point>

File: interface_description/urdf/usb30.urdf.xacro (robot description, xacro)
@@ -1,4 +1,5 @@
 <?xml version="1.0" encoding="UTF-8" ?>
 <robot xmlns:xacro="http://ros.org/wiki/xacro"
+       xmlns:usb="urn:ietf:params:xml:ns:yang:usb-port"
        name="usb30">
     <xacro:macro name="usb30" params="parent prefix id:=0 origin_xyz origin_rpy">
@@ -27,13 +28,12 @@
         <nt:termination-point xmlns:nt="urn:ietf:params:xml:ns:yang:ietf-network-topology">
             <nt:tp-id>${prefix}-usb30-${id}</nt:tp-id>
-            <dl:device-layer-termination-point-attributes xmlns:dl="urn:ietf:params:xml:ns:yang:device-layer">
-                <dl:port-name>usb30-${id}</dl:port-name>
+            <dl:device-layer-termination-point-attributes
+                xmlns:dl="urn:ietf:params:xml:ns:yang:device-layer"
+                xmlns:usb="urn:ietf:params:xml:ns:yang:usb-port">
+                <dl:port-name>${prefix}-usb30</dl:port-name>
                 <dl:port-type>usb</dl:port-type>
-                <usb:usb-port xmlns:usb="urn:ietf:params:xml:ns:yang:usb-port">
-                    <usb:port-id>${prefix}-usb30-${id}</usb:port-id>
-                    <usb:version>usb3.0</usb:version>
-                    <usb:speed>5.00</usb:speed>
-                    <usb:power-consumption>2.5</usb:power-consumption>
-                </usb:usb-port>
+                <dl:wired>true</dl:wired>
+                <usb:version>usb3.0</usb:version>
+                <usb:power-consumption>2.5</usb:power-consumption>
             </dl:device-layer-termination-point-attributes>
         </nt:termination-point>

Commit message: xml namespace added

File: interface_description/urdf/cat5e.urdf.xacro (robot description, xacro)
@@ -2,5 +2,6 @@
 <robot xmlns:xacro="http://ros.org/wiki/xacro"
        name="cat5e">
-    <xacro:macro name="cat5e" params="parent prefix id:=0 origin_xyz origin_rpy">
+    <xacro:macro name="cat5e" params="parent prefix id:=0 origin_xyz origin_rpy"
+        xmlns:nt="urn:ietf:params:xml:ns:yang:ietf-network-topology">
         <joint name="${prefix}-cat5e-${id}-joint" type="fixed">
             <origin xyz="${origin_xyz}" rpy="${origin_rpy}" />

File: interface_description/urdf/cat6.urdf.xacro (robot description, xacro)
@@ -1,6 +1,8 @@
 <?xml version="1.0" encoding="UTF-8" ?>
 <robot xmlns:xacro="http://ros.org/wiki/xacro"
+       xmlns:nt="urn:ietf:params:xml:ns:yang:ietf-network-topology"
        name="cat6">
-    <xacro:macro name="cat6" params="parent prefix id:=0 origin_xyz origin_rpy">
+    <xacro:macro name="cat6" params="parent prefix id:=0 origin_xyz origin_rpy"
+        xmlns:nt="urn:ietf:params:xml:ns:yang:ietf-network-topology">
         <joint name="${prefix}-cat6-${id}-joint" type="fixed">
             <origin xyz="${origin_xyz}" rpy="${origin_rpy}" />

File: interface_description/urdf/usb-typec.urdf.xacro (robot description, xacro)
@@ -3,5 +3,6 @@
        xmlns:usb="urn:ietf:params:xml:ns:yang:usb-port"
        name="usb_typec">
-    <xacro:macro name="usb_typec" params="parent prefix id:=0 origin_xyz origin_rpy">
+    <xacro:macro name="usb_typec" params="parent prefix id:=0 origin_xyz origin_rpy"
+        xmlns:nt="urn:ietf:params:xml:ns:yang:ietf-network-topology">
         <joint name="${prefix}-usb-typec-${id}-joint" type="fixed">
             <origin xyz="${origin_xyz}" rpy="${origin_rpy}" />

File: interface_description/urdf/usb20.urdf.xacro (robot description, xacro)
@@ -3,5 +3,6 @@
        xmlns:usb="urn:ietf:params:xml:ns:yang:usb-port"
        name="usb20">
-    <xacro:macro name="usb20" params="parent prefix id:=0 origin_xyz origin_rpy">
+    <xacro:macro name="usb20" params="parent prefix id:=0 origin_xyz origin_rpy"
+        xmlns:nt="urn:ietf:params:xml:ns:yang:ietf-network-topology">
         <joint name="${prefix}-usb20-${id}-joint" type="fixed">
             <origin xyz="${origin_xyz}" rpy="${origin_rpy}" />

File: interface_description/urdf/usb30.urdf.xacro (robot description, xacro)
@@ -3,5 +3,6 @@
        xmlns:usb="urn:ietf:params:xml:ns:yang:usb-port"
        name="usb30">
-    <xacro:macro name="usb30" params="parent prefix id:=0 origin_xyz origin_rpy">
+    <xacro:macro name="usb30" params="parent prefix id:=0 origin_xyz origin_rpy"
+        xmlns:nt="urn:ietf:params:xml:ns:yang:ietf-network-topology">
         <joint name="${prefix}-usb30-${id}-joint" type="fixed">
             <origin xyz="${origin_xyz}" rpy="${origin_rpy}" />
