Commit message: ports & yangs updated

File: nuc_description/urdf/nuc.urdf.xacro (robot description, xacro)
@@ -4,7 +4,7 @@
     <xacro:include filename="$(find interface_description)/urdf/cat6.urdf.xacro"/>
     <xacro:include filename="$(find interface_description)/urdf/usb30.urdf.xacro"/>
-    <xacro:include filename="$(find interface_description)/urdf/wifi4.urdf.xacro"/>
-    <xacro:include filename="$(find interface_description)/urdf/wifi5.urdf.xacro"/>
-    <xacro:macro name="nuc" params="parent id xyz:= '-1 1 0' L2_network_id:=nuc_network_level L1_network_id:=nuc_device_level L2_id:=nuc_L2 L1_id:=nuc_L1">
+    <!-- <xacro:include filename="$(find interface_description)/urdf/wifi4.urdf.xacro"/> -->
+    <!-- <xacro:include filename="$(find interface_description)/urdf/wifi5.urdf.xacro"/> -->
+    <xacro:macro name="nuc" params="parent id:=0 xyz:= '-1 1 0' ">
         <joint name="nuc_${id}_joint" type="fixed">
             <origin xyz="${xyz}" rpy="0 0 0" />
@@ -37,16 +37,16 @@
         </joint>
         <link name="nuc_${id}_rj45_0_link">
-        <visual>
-            <origin xyz="0 0 0" rpy="0 0 0"/>
-            <geometry>
-            <mesh filename="file://$(find interface_description)/meshes/rj45-female.stl" scale="0.001 0.001 0.001" />
-            </geometry>
-        </visual>
-        <collision>
-            <origin xyz="0 0 0" rpy="0 0 0"/>
-            <geometry>
-            <mesh filename="file://$(find interface_description)/meshes/rj45-female.stl" scale="0.001 0.001 0.001" />
-            </geometry>
-        </collision>
+            <visual>
+                <origin xyz="0 0 0" rpy="0 0 0"/>
+                <geometry>
+                <mesh filename="file://$(find interface_description)/meshes/rj45-female.stl" scale="0.001 0.001 0.001" />
+                </geometry>
+            </visual>
+            <collision>
+                <origin xyz="0 0 0" rpy="0 0 0"/>
+                <geometry>
+                <mesh filename="file://$(find interface_description)/meshes/rj45-female.stl" scale="0.001 0.001 0.001" />
+                </geometry>
+            </collision>
         </link>
         <!-- USB-30-0 -->
@@ -57,16 +57,16 @@
         </joint>
         <link name="nuc_${id}_usb-a-30_0_link">
-        <visual>
-            <origin xyz="0 0 0" rpy="0 0 0"/>
-            <geometry>
-            <mesh filename="file://$(find interface_description)/meshes/usb-A-female.stl" scale="0.001 0.001 0.001" />
-            </geometry>
-        </visual>
-        <collision>
-            <origin xyz="0 0 0" rpy="0 0 0"/>
-            <geometry>
-            <mesh filename="file://$(find interface_description)/meshes/usb-A-female.stl" scale="0.001 0.001 0.001" />
-            </geometry>
-        </collision>
+            <visual>
+                <origin xyz="0 0 0" rpy="0 0 0"/>
+                <geometry>
+                <mesh filename="file://$(find interface_description)/meshes/usb-A-female.stl" scale="0.001 0.001 0.001" />
+                </geometry>
+            </visual>
+            <collision>
+                <origin xyz="0 0 0" rpy="0 0 0"/>
+                <geometry>
+                <mesh filename="file://$(find interface_description)/meshes/usb-A-female.stl" scale="0.001 0.001 0.001" />
+                </geometry>
+            </collision>
         </link>
         <!-- USB-30-1 -->
@@ -77,91 +77,45 @@
         </joint>
         <link name="nuc_${id}_usb-a-30_1_link">
-        <visual>
-            <origin xyz="0 0 0" rpy="0 0 0"/>
-            <geometry>
-            <mesh filename="file://$(find interface_description)/meshes/usb-A-female.stl" scale="0.001 0.001 0.001" />
-            </geometry>
-        </visual>
-        <collision>
-            <origin xyz="0 0 0" rpy="0 0 0"/>
-            <geometry>
-            <mesh filename="file://$(find interface_description)/meshes/usb-A-female.stl" scale="0.001 0.001 0.001" />
-            </geometry>
-        </collision>
+            <visual>
+                <origin xyz="0 0 0" rpy="0 0 0"/>
+                <geometry>
+                <mesh filename="file://$(find interface_description)/meshes/usb-A-female.stl" scale="0.001 0.001 0.001" />
+                </geometry>
+            </visual>
+            <collision>
+                <origin xyz="0 0 0" rpy="0 0 0"/>
+                <geometry>
+                <mesh filename="file://$(find interface_description)/meshes/usb-A-female.stl" scale="0.001 0.001 0.001" />
+                </geometry>
+            </collision>
         </link>
         <yang>
             <!-- NUC network topology -->
+            <!-- valahol ezen belül példányosítani kell az usb-t! -->
+            <!-- <xacro:usb30 parent="world" id="0"> -->
             <network>
-                <network-id>${L2_network_id}</network-id>
+                <network-id>nuc-network</network-id>
+                <network-types>
+                    <dl:device-layer-topology xmlns:dl="urn:ietf:params:xml:ns:yang:device-layer"/>
+                </network-types>
                 <supporting-network>
-                    <network-ref>${L1_network_id}</network-ref>
+                    <network-ref>nuc-supporting-network</network-ref>
                 </supporting-network>
                 <node>
-                <node-id>${L2_id}</node-id>
-                <supporting-node>
-                    <network-ref>${L1_network_id}</network-ref>
-                    <node-ref>${L1_id}</node-ref>
-                </supporting-node>
-                <dl:device-layer-node-attributes xmlns:dl="urn:ietf:params:xml:ns:yang:device-layer">
-                    <dl:device-name>NUC</dl:device-name>
-                    <dl:device-type>pc</dl:device-type>
-                </dl:device-layer-node-attributes>
-                <nt:termination-point xmlns:nt="urn:ietf:params:xml:ns:yang:ietf-network-topology">
-                    <nt:tp-id>_0</nt:tp-id>
-                    <nt:supporting-termination-point>
-                        <nt:network-ref>${L2_id}</nt:network-ref>
-                        <nt:node-ref>${L1_id}</nt:node-ref>
-                        <nt:tp-ref>eth_0</nt:tp-ref>
-                    </nt:supporting-termination-point>
-                    <dl:device-layer-termination-point-attributes xmlns:dl="urn:ietf:params:xml:ns:yang:device-layer">
-                        <dl:port-name>port1</dl:port-name>
-                        <dl:port-type>rj45</dl:port-type>
-                    </dl:device-layer-termination-point-attributes>
-                    <nl:network-layer-termination-point-attributes xmlns:nl="urn:ietf:params:xml:ns:yang:network-layer">
-                        <nl:interface-name>intf1</nl:interface-name>
-                        <nl:interface-type>ethernet</nl:interface-type>
-                        <nl:interface-status>up</nl:interface-status>
-                        <nl:mac-address>00:1A:2B:3C:4D:5E</nl:mac-address>
-                    </nl:network-layer-termination-point-attributes>
-                </nt:termination-point>
-                <nl:network-layer-node-attributes xmlns:nl="urn:ietf:params:xml:ns:yang:network-layer">
-                    <nl:node-name>netNode1</nl:node-name>
-                    <nl:node-type>generic</nl:node-type>
-                </nl:network-layer-node-attributes>
+                    <node-id>nuc-usb-node</node-id>
+                    <supporting-node>
+                        <network-ref>nuc-usb-supporting-network</network-ref>
+                        <node-ref>nuc-usb-supporting-node</node-ref>
+                    </supporting-node>
+                    <xacro:usb30 parent="world" id="0" />
                 </node>
-                <dl:device-layer-topology xmlns:dl="urn:ietf:params:xml:ns:yang:device-layer">
-                    <dl:element>element2</dl:element>
-                </dl:device-layer-topology>
-                <nt:link xmlns:nt="urn:ietf:params:xml:ns:yang:ietf-network-topology">
-                    <nt:link-id>link1</nt:link-id>
-                    <nt:source>
-                        <nt:source-node>node1</nt:source-node>
-                        <nt:source-tp>tp1</nt:source-tp>
-                    </nt:source>
-                    <nt:destination>
-                        <nt:dest-node>node2</nt:dest-node>
-                        <nt:dest-tp>tp2</nt:dest-tp>
-                    </nt:destination>
-                    <nt:supporting-link>
-                        <nt:network-ref>network2</nt:network-ref>
-                        <nt:link-ref>link2</nt:link-ref>
-                    </nt:supporting-link>
-                    <dl:device-layer-link-attributes xmlns:dl="urn:ietf:params:xml:ns:yang:device-layer">
-                        <dl:physical-link-name>physLink1</dl:physical-link-name>
-                        <dl:physical-link-type>cat5e</dl:physical-link-type>
-                    </dl:device-layer-link-attributes>
-                    <nl:network-layer-link-attributes xmlns:nl="urn:ietf:params:xml:ns:yang:network-layer">
-                        <nl:link-name>netLink1</nl:link-name>
-                        <nl:link-type>3gpp-5g-qos-flow</nl:link-type>
-                        <nl:_5qi>1</nl:_5qi>
-                        <nl:gfbr>50</nl:gfbr>
-                        <nl:mfbr>100</nl:mfbr>
-                        <nl:pdb>20</nl:pdb>
-                        <nl:per>0</nl:per>
-                    </nl:network-layer-link-attributes>
-                </nt:link>
-                <nl:network-layer-topology xmlns:nl="urn:ietf:params:xml:ns:yang:network-layer">
-                    <nl:element>element3</nl:element>
-                </nl:network-layer-topology>
+                <node>
+                    <node-id>nuc-cat6-node</node-id>
+                    <supporting-node>
+                        <network-ref>nuc-cat6-supporting-network</network-ref>
+                        <node-ref>nuc-cat6-supporting-node</node-ref>
+                    </supporting-node>
+                    <xacro:cat6 parent="world" id="0" />
+                </node>
             </network>
         </yang>

Commit message: yang content update

File: nuc_description/urdf/nuc.urdf.xacro (robot description, xacro)
@@ -4,12 +4,12 @@
     <xacro:include filename="$(find interface_description)/urdf/cat6.urdf.xacro"/>
     <xacro:include filename="$(find interface_description)/urdf/usb30.urdf.xacro"/>
-    <xacro:macro name="nuc" params="parent id:=0 xyz:='-1 1 0' ">
-        <joint name="nuc_${id}_joint" type="fixed">
-            <origin xyz="${xyz}" rpy="0 0 0" />
+    <xacro:macro name="nuc" params="parent id:=0 origin_xyz:='-1 1 0' ">
+        <joint name="nuc-${id}-joint" type="fixed">
+            <origin xyz="${origin_xyz}" rpy="0 0 0" />
             <!-- <origin xyz="-1 1 0" rpy="0 0 0" /> -->
             <parent link="${parent}"/>
-            <child link="nuc_${id}_link"/>
+            <child link="nuc-${id}-link"/>
         </joint>
-        <link name="nuc_${id}_link">
+        <link name="nuc-${id}-link">
             <visual>
                 <origin rpy="0 0 0" xyz="0 0 0"/>
@@ -28,68 +28,9 @@
             </collision>
         </link>
-        <!-- ethernet-0 -->
-        <joint name="nuc_${id}_rj45_0_frame" type="fixed">
-            <parent link="nuc_${id}_link"/>
-            <child link="nuc_${id}_rj45_0_link"/>
-            <origin xyz="0.04 0.068 0.032" rpy="-1.5707963 0 0"/>
-        </joint>
-        <link name="nuc_${id}_rj45_0_link">
-            <visual>
-                <origin xyz="0 0 0" rpy="0 0 0"/>
-                <geometry>
-                <mesh filename="file://$(find interface_description)/meshes/rj45-female.stl" scale="0.001 0.001 0.001" />
-                </geometry>
-            </visual>
-            <collision>
-                <origin xyz="0 0 0" rpy="0 0 0"/>
-                <geometry>
-                <mesh filename="file://$(find interface_description)/meshes/rj45-female.stl" scale="0.001 0.001 0.001" />
-                </geometry>
-            </collision>
-        </link>
-        <!-- USB-30-0 -->
-        <joint name="nuc_${id}_usb-a-30_0_frame" type="fixed">
-            <parent link="nuc_${id}_link"/>
-            <child link="nuc_${id}_usb-a-30_0_link"/>
-            <origin xyz="0.087 0.119 0.019" rpy="1.5707963 1.5707963 0"/>
-        </joint>
-        <link name="nuc_${id}_usb-a-30_0_link">
-            <visual>
-                <origin xyz="0 0 0" rpy="0 0 0"/>
-                <geometry>
-                <mesh filename="file://$(find interface_description)/meshes/usb-A-female.stl" scale="0.001 0.001 0.001" />
-                </geometry>
-            </visual>
-            <collision>
-                <origin xyz="0 0 0" rpy="0 0 0"/>
-                <geometry>
-                <mesh filename="file://$(find interface_description)/meshes/usb-A-female.stl" scale="0.001 0.001 0.001" />
-                </geometry>
-            </collision>
-        </link>
-        <!-- USB-30-1 -->
-        <joint name="nuc_${id}_usb-a-30_1_frame" type="fixed">
-            <parent link="nuc_${id}_link"/>
-            <child link="nuc_${id}_usb-a-30_1_link"/>
-            <origin xyz="0.075 0.119 0.019" rpy="1.5707963 1.5707963 0"/>
-        </joint>
-        <link name="nuc_${id}_usb-a-30_1_link">
-            <visual>
-                <origin xyz="0 0 0" rpy="0 0 0"/>
-                <geometry>
-                <mesh filename="file://$(find interface_description)/meshes/usb-A-female.stl" scale="0.001 0.001 0.001" />
-                </geometry>
-            </visual>
-            <collision>
-                <origin xyz="0 0 0" rpy="0 0 0"/>
-                <geometry>
-                <mesh filename="file://$(find interface_description)/meshes/usb-A-female.stl" scale="0.001 0.001 0.001" />
-                </geometry>
-            </collision>
-        </link>
         <!-- NUC network topology -->
         <node>
             <node-id>nuc-${id}-usb-node</node-id>
-            <xacro:usb30 parent="world" id="0" />
+            <xacro:usb30 parent="nuc-${id}-link" prefix="nuc-${id}" id="0" origin_xyz="0.087 0.119 0.019" origin_rpy="1.57 1.57 0"/>
+            <xacro:usb30 parent="nuc-${id}-link" prefix="nuc-${id}" id="1" origin_xyz="0.075 0.119 0.0199" origin_rpy="1.57 1.57 0"/>
         </node>
         <node>
@@ -99,5 +40,5 @@
                 <dl:device-type>pc</dl:device-type>
             </dl:device-layer-node-attributes>
-            <xacro:cat6 parent="world" id="0" />
+            <xacro:cat6 parent="nuc-${id}-link" prefix="nuc-${id}" id="0" origin_xyz="0.04 0.068 0.032" origin_rpy="-1.5707963 0 0"/>
         </node>
     </xacro:macro>

Commit message: attribs updated

File: nuc_description/urdf/nuc.urdf.xacro (robot description, xacro)
@@ -4,8 +4,7 @@
     <xacro:include filename="$(find interface_description)/urdf/cat6.urdf.xacro"/>
     <xacro:include filename="$(find interface_description)/urdf/usb30.urdf.xacro"/>
-    <xacro:macro name="nuc" params="parent id:=0 origin_xyz:='-1 1 0' ">
+    <xacro:macro name="nuc" params="parent id:=0 origin_xyz:='-1 1 0' origin_rpy:='0 0 0' ">
         <joint name="nuc-${id}-joint" type="fixed">
-            <origin xyz="${origin_xyz}" rpy="0 0 0" />
-            <!-- <origin xyz="-1 1 0" rpy="0 0 0" /> -->
+            <origin xyz="${origin_xyz}" rpy="${origin_rpy}" />
             <parent link="${parent}"/>
             <child link="nuc-${id}-link"/>
@@ -30,10 +29,5 @@
         <!-- NUC network topology -->
         <node>
-            <node-id>nuc-${id}-usb-node</node-id>
-            <xacro:usb30 parent="nuc-${id}-link" prefix="nuc-${id}" id="0" origin_xyz="0.087 0.119 0.019" origin_rpy="1.57 1.57 0"/>
-            <xacro:usb30 parent="nuc-${id}-link" prefix="nuc-${id}" id="1" origin_xyz="0.075 0.119 0.0199" origin_rpy="1.57 1.57 0"/>
-        </node>
-        <node>
-            <node-id>nuc-${id}-cat6-node</node-id>
+            <node-id>nuc-${id}-node</node-id>
             <dl:device-layer-node-attributes xmlns:dl="urn:ietf:params:xml:ns:yang:device-layer">
                 <dl:device-name>nuc-${id}</dl:device-name>
@@ -41,4 +35,6 @@
             </dl:device-layer-node-attributes>
             <xacro:cat6 parent="nuc-${id}-link" prefix="nuc-${id}" id="0" origin_xyz="0.04 0.068 0.032" origin_rpy="-1.5707963 0 0"/>
+            <xacro:usb30 parent="nuc-${id}-link" prefix="nuc-${id}" id="0" origin_xyz="0.087 0.119 0.019" origin_rpy="1.57 1.57 0"/>
+            <xacro:usb30 parent="nuc-${id}-link" prefix="nuc-${id}" id="1" origin_xyz="0.075 0.119 0.0199" origin_rpy="1.57 1.57 0"/>
         </node>
     </xacro:macro>
