Commit message: progress

File: cable_description/urdf/ethernet-cable.urdf.xacro (robot description, xacro)
@@ -1,10 +1,9 @@
 <?xml version="1.0"?>
-<robot name="ethernet-cable"
-    xmlns:xacro="http://wiki.ros.org/xacro">
-    <xacro:macro name="ethernet-cable" params="parent src_port dst_port length src_node:=camera-0 src_tp:=usb-typec-0 dst_node:=d455 dst_tp:=usb30-0 link_type:=usb30 length:=2">
-                                                        <!-- biztos h port?? tp és node alapján adom meg! -->
+<robot xmlns:xacro="http://wiki.ros.org/xacro"
+       name="eth-cable">
+    <xacro:macro name="eth-cable" params="parent src_node:='camera-0' src_tp:='usb-typec-0' dst_node:='d455' dst_tp:='usb30-0' link_type:='usb30' length:='2'">
         <joint name="ethernet-cable-joint" type="fixed">
             <origin xyz="0 0 0" rpy="0 0 0"/>
-            <parent link="${src_port}"/>
+            <parent link="${parent}"/>
             <child link="ethernet-cable-link"/> <!-- kábel csonk -->
         </joint>
@@ -41,5 +40,5 @@
                 <dl:physical-link-name>${src_node}-${dst_node}-cable</dl:physical-link-name>
                 <dl:physical-link-type>${link_type}</dl:physical-link-type>
-                <dl:cable-length>${length}</dl:cable-length>
+                <dl:cable-length>2</dl:cable-length>
             </dl:device-layer-link-attributes>
         </nt:link>

Commit message: general cable urdf

File: cable_description/urdf/ethernet-cable.urdf.xacro (robot description, xacro)
@@ -2,5 +2,5 @@
 <robot xmlns:xacro="http://wiki.ros.org/xacro"
        name="eth-cable">
-    <xacro:macro name="eth-cable" params="parent src_node:='camera-0' src_tp:='usb-typec-0' dst_node:='d455' dst_tp:='usb30-0' link_type:='usb30' length:='2'">
+    <xacro:macro name="eth-cable" params="parent src_node dst_node src_tp dst_tp link_type">
         <joint name="ethernet-cable-joint" type="fixed">
             <origin xyz="0 0 0" rpy="0 0 0"/>
@@ -12,5 +12,5 @@
                 <origin rpy="0 0 0" xyz="0 0 0"/>
                 <geometry>
-                    <cylinder length="${length}" radius="0.001"/> <!-- measure 3D point distances -->
+                    <cylinder length="2" radius="0.001"/> <!-- measure 3D point distances -->
                 </geometry>
                 <material name="Black">
@@ -21,5 +21,5 @@
                 <origin xyz="0 0 0" rpy="0 0 0"/>
                 <geometry>
-                    <cylinder length="${length}" radius="0.001"/>
+                    <cylinder length="2" radius="0.001"/>
                 </geometry>
             </collision>

Commit message: length as arg added

File: cable_description/urdf/ethernet-cable.urdf.xacro (robot description, xacro)
@@ -2,5 +2,5 @@
 <robot xmlns:xacro="http://wiki.ros.org/xacro"
        name="eth-cable">
-    <xacro:macro name="eth-cable" params="parent src_node dst_node src_tp dst_tp link_type">
+    <xacro:macro name="eth-cable" params="parent src_node dst_node src_tp dst_tp link_type length">
         <joint name="ethernet-cable-joint" type="fixed">
             <origin xyz="0 0 0" rpy="0 0 0"/>
@@ -12,5 +12,5 @@
                 <origin rpy="0 0 0" xyz="0 0 0"/>
                 <geometry>
-                    <cylinder length="2" radius="0.001"/> <!-- measure 3D point distances -->
+                    <cylinder length="${length}" radius="0.001"/> <!-- measure 3D point distances -->
                 </geometry>
                 <material name="Black">
@@ -21,5 +21,5 @@
                 <origin xyz="0 0 0" rpy="0 0 0"/>
                 <geometry>
-                    <cylinder length="2" radius="0.001"/>
+                    <cylinder length="${length}" radius="0.001"/>
                 </geometry>
             </collision>
@@ -40,5 +40,5 @@
                 <dl:physical-link-name>${src_node}-${dst_node}-cable</dl:physical-link-name>
                 <dl:physical-link-type>${link_type}</dl:physical-link-type>
-                <dl:cable-length>2</dl:cable-length>
+                <dl:cable-length>${length}</dl:cable-length>
             </dl:device-layer-link-attributes>
         </nt:link>

File: cable_description/urdf/usb-cable.urdf.xacro (robot description, xacro)
@@ -1,9 +1,9 @@
 <?xml version="1.0"?>
-<robot name="usb-cable"
-    xmlns:xacro="http://wiki.ros.org/xacro">
-    <xacro:macro name="usb-cable" params="parent src_port dst_port length">
+<robot xmlns:xacro="http://wiki.ros.org/xacro"
+       name="usb-cable">
+    <xacro:macro name="usb-cable" params="parent src_node dst_node src_tp dst_tp link_type length">
         <joint name="usb-cable-joint" type="fixed">
             <origin xyz="0 0 0" rpy="0 0 0"/>
-            <parent link="${src_port}"/>
+            <parent link="${parent}"/>
             <child link="usb-cable-link"/> <!-- kábel csonk -->
         </joint>
@@ -25,13 +25,14 @@
             </collision>
         </link>
-        <!-- <nt:link xmlns:nt="urn:ietf:params:xml:ns:yang:ietf-network-topology">
-            <nt:link-id>${src_port}-${dst_port}-link</nt:link-id>
+        <!-- todo: dugo tipust kivlasztani mesh-bol -->
+        <nt:link xmlns:nt="urn:ietf:params:xml:ns:yang:ietf-network-topology">
+            <nt:link-id>${src_node}-${dst_node}-link</nt:link-id>
             <nt:source>
-                <nt:source-node>${src_port}</nt:source-node>
-                <nt:source-tp>${src_port}-usb30-${src_port}</nt:source-tp>
+                <nt:source-node>${src_node}</nt:source-node>
+                <nt:source-tp>${src_node}-${src_tp}</nt:source-tp>
             </nt:source>
             <nt:destination>
-                <nt:dest-node>${dst_port}</nt:dest-node>
-                <nt:dest-tp>${dst_port}-usb30-${dst_port}</nt:dest-tp>
+                <nt:dest-node>${dst_node}</nt:dest-node>
+                <nt:dest-tp>${dst_node}-${dst_tp}</nt:dest-tp>
             </nt:destination>
             <dl:device-layer-link-attributes
@@ -41,5 +42,10 @@
                 <dl:physical-link-type>usb30</dl:physical-link-type>
                 <dl:cable-length>${length}</dl:cable-length>
-                <usb:source-connector-type       -->
+                <usb:source-connector-type>usb30</usb:source-connector-type>
+                <usb:destination-connector-type>usb30</usb:destination-connector-type>
+                <usb:max-data-transfer>20</usb:max-data-transfer>
+                <usb:max-power-transfer>150</usb:max-power-transfer>
+            </dl:device-layer-link-attributes>
+        </nt:link>
     </xacro:macro>
 </robot>

Commit message: fixed

File: cable_description/urdf/ethernet-cable.urdf.xacro (robot description, xacro)
@@ -1,6 +1,6 @@
 <?xml version="1.0"?>
 <robot xmlns:xacro="http://wiki.ros.org/xacro"
-       name="eth-cable">
-    <xacro:macro name="eth-cable" params="parent src_node dst_node src_tp dst_tp link_type length">
+       name="ethernet-cable">
+    <xacro:macro name="ethernet-cable" params="parent src_node dst_node src_tp dst_tp link_type length">
         <joint name="ethernet-cable-joint" type="fixed">
             <origin xyz="0 0 0" rpy="0 0 0"/>
@@ -25,5 +25,4 @@
             </collision>
         </link>
-        <!-- todo: dugo tipust kivlasztani mesh-bol -->
         <nt:link xmlns:nt="urn:ietf:params:xml:ns:yang:ietf-network-topology">
             <nt:link-id>${src_node}-${dst_node}-link</nt:link-id>

File: cable_description/urdf/usb-cable.urdf.xacro (robot description, xacro)
@@ -25,5 +25,4 @@
             </collision>
         </link>
-        <!-- todo: dugo tipust kivlasztani mesh-bol -->
         <nt:link xmlns:nt="urn:ietf:params:xml:ns:yang:ietf-network-topology">
             <nt:link-id>${src_node}-${dst_node}-link</nt:link-id>
