Commit message: config updated

File: example_config/urdf/system_config.urdf.xacro (robot description, xacro)
@@ -12,7 +12,7 @@
     <!-- import d455 camera -->
     <xacro:include filename="$(find realsense2_description)/urdf/_d455.urdf.xacro" />
-    <xacro:sensor_d455 parent="world">
+    <!-- <xacro:sensor_d455 parent="world">
         <origin xyz="-0.022 -0.039 -0.01" rpy="0 1.57 0" />
-    </xacro:sensor_d455>
+    </xacro:sensor_d455> -->
     <xacro:nuc parent="world" id="0" />
 </robot>

File: interface_description/urdf/cat6.urdf.xacro (robot description, xacro)
@@ -6,10 +6,10 @@
        name="cat6">
     <xacro:macro name="cat6" params="parent id:=0">
-        <joint name="cat6_joint" type="fixed">
+        <joint name="cat6-${id}_joint" type="fixed">
             <origin xyz="-1 1 0" rpy="0 0 0" />
             <parent link="${parent}"/>
-            <child link="cat6_link"/>
+            <child link="cat6-${id}_link"/>
         </joint>
-        <link name="cat6_link">
+        <link name="cat6-${id}_link">
             <visual>
                 <origin rpy="0 0 0" xyz="0 0 0"/>
@@ -31,19 +31,19 @@
             <!-- cat6 network topology -->
             <network>
-                <network-id>cat6-network</network-id>
+                <network-id>cat6-${id}-network</network-id>
                 <network-types>
                     <dl:device-layer-topology xmlns:dl="urn:ietf:params:xml:ns:yang:device-layer"/>
                 </network-types>
                 <supporting-network>
-                    <network-ref>cat6-supporting-network</network-ref>
+                    <network-ref>cat6-${id}-supporting-network</network-ref>
                 </supporting-network>
                 <node>
-                    <node-id>cat6-node</node-id>
+                    <node-id>cat6-${id}-node</node-id>
                     <supporting-node>
-                        <network-ref>cat6-supporting-network</network-ref>
-                        <node-ref>cat6-supporting-node</node-ref>
+                        <network-ref>cat6-${id}-supporting-network</network-ref>
+                        <node-ref>cat6-${id}-supporting-node</node-ref>
                     </supporting-node>
                     <dl:device-layer-node-attributes xmlns:dl="urn:ietf:params:xml:ns:yang:device-layer">
-                        <dl:device-name>cat6-interface</dl:device-name>
+                        <dl:device-name>cat6-${id}-interface</dl:device-name>
                         <dl:device-type>port</dl:device-type>
                     </dl:device-layer-node-attributes>
@@ -56,8 +56,8 @@
                         </nt:supporting-termination-point>
                         <dl:device-layer-termination-point-attributes xmlns:dl="urn:ietf:params:xml:ns:yang:device-layer">
-                            <dl:port-name>port-1</dl:port-name>
+                            <dl:port-name>rj45-${id}</dl:port-name>
                             <dl:port-type>
                                 <eth:ethernet-port xmlns:eth="urn:ietf:params:xml:ns:yang:ethernet-port">
-                                <eth:port-id>eth1</eth:port-id>
+                                <eth:port-id>eth-${id}</eth:port-id>
                                 <eth:mac-address>00:1A:2B:3C:4D:5E</eth:mac-address>
                                 <eth:speed>1000Mbps</eth:speed>

File: interface_description/urdf/usb-typec.urdf.xacro (robot description, xacro)
@@ -5,11 +5,11 @@
        xmlns:usb-port="urn:ietf:params:xml:ns:yang:usb-port"
        name="usb_typec">
-    <xacro:macro name="usb_typec" params="parent">
-        <joint name="usb_typec_joint" type="fixed">
+    <xacro:macro name="usb_typec" params="parent id=0">
+        <joint name="usb-typec-${id}_joint" type="fixed">
             <origin xyz="-1 1 0" rpy="0 0 0" />
             <parent link="${parent}"/>
-            <child link="usb-typec_link"/>
+            <child link="usb-typec-${id}_link"/>
         </joint>
-        <link name="usb_typec_link">
+        <link name="usb-typec-${id}_link">
             <visual>
                 <origin rpy="0 0 0" xyz="0 0 0"/>
@@ -31,20 +31,20 @@
             <!-- usb-typec network topology -->
             <network>
-                <network-id>usb-typec-network</network-id>
+                <network-id>usb-typec-${id}-network</network-id>
                 <network-types>
                     <dl:device-layer-topology xmlns:dl="urn:ietf:params:xml:ns:yang:device-layer"/>
                 </network-types>
                 <supporting-network>
-                    <network-ref>usb-typec-supporting-network</network-ref>
+                    <network-ref>usb-typec-${id}-supporting-network</network-ref>
                 </supporting-network>
                 <node>
-                    <node-id>usb-typec-node</node-id>
+                    <node-id>usb-typec-${id}-node</node-id>
                     <supporting-node>
-                        <network-ref>usb-typec-supporting-network</network-ref>
-                        <node-ref>usb-typec-supporting-node</node-ref>
+                        <network-ref>usb-typec-${id}-supporting-network</network-ref>
+                        <node-ref>usb-typec-${id}-supporting-node</node-ref>
                     </supporting-node>
                     <dl:device-layer-node-attributes xmlns:dl="urn:ietf:params:xml:ns:yang:device-layer">
-                        <dl:device-name>usb-typec-device</dl:device-name>
-                        <dl:device-type>usb-typec-port</dl:device-type>
+                        <dl:device-name>usb-typec-${id}-device</dl:device-name>
+                        <dl:device-type>usb-typec-${id}-port</dl:device-type>
                     </dl:device-layer-node-attributes>
                     <nt:termination-point xmlns:nt="urn:ietf:params:xml:ns:yang:ietf-network-topology">
@@ -59,5 +59,5 @@
                             <dl:port-type>
                                 <usb:usb-port xmlns:usb="urn:ietf:params:xml:ns:yang:usb-port">
-                                <usb:port-id>usb-typec</usb:port-id>
+                                <usb:port-id>usb-typec-${id}</usb:port-id>
                                 <usb:version>USB3.2</usb:version>
                                 <usb:speed>5.00</usb:speed>

File: interface_description/urdf/usb30.urdf.xacro (robot description, xacro)
@@ -6,10 +6,10 @@
        name="usb30">
     <xacro:macro name="usb30" params="parent id:=0">
-        <joint name="usb30_joint" type="fixed">
+        <joint name="usb30-${id}_joint" type="fixed">
             <origin xyz="-1 1 0" rpy="0 0 0" />
             <parent link="${parent}"/>
-            <child link="usb30_link"/>
+            <child link="usb30-${id}_link"/>
         </joint>
-        <link name="usb30_link">
+        <link name="usb30-${id}_link">
             <visual>
                 <origin rpy="0 0 0" xyz="0 0 0"/>
@@ -31,20 +31,20 @@
             <!-- usb30 network topology -->
             <network>
-                <network-id>usb30-network</network-id>
+                <network-id>usb30-${id}-network</network-id>
                 <network-types>
                     <dl:device-layer-topology xmlns:dl="urn:ietf:params:xml:ns:yang:device-layer"/>
                 </network-types>
                 <supporting-network>
-                    <network-ref>usb30-supporting-network</network-ref>
+                    <network-ref>usb30-${id}-supporting-network</network-ref>
                 </supporting-network>
                 <node>
-                    <node-id>usb30-node</node-id>
+                    <node-id>usb30-${id}-node</node-id>
                     <supporting-node>
-                        <network-ref>usb30-supporting-network</network-ref>
-                        <node-ref>usb30-supporting-node</node-ref>
+                        <network-ref>usb30-${id}-supporting-network</network-ref>
+                        <node-ref>usb30-${id}-supporting-node</node-ref>
                     </supporting-node>
                     <dl:device-layer-node-attributes xmlns:dl="urn:ietf:params:xml:ns:yang:device-layer">
-                        <dl:device-name>usb30-device</dl:device-name>
-                        <dl:device-type>usb30-port</dl:device-type>
+                        <dl:device-name>usb30-${id}-device</dl:device-name>
+                        <dl:device-type>usb30-${id}-port</dl:device-type>
                     </dl:device-layer-node-attributes>
                     <nt:termination-point xmlns:nt="urn:ietf:params:xml:ns:yang:ietf-network-topology">
@@ -59,5 +59,5 @@
                             <dl:port-type>
                                 <usb:usb-port xmlns:usb="urn:ietf:params:xml:ns:yang:usb-port">
-                                <usb:port-id>eth1</usb:port-id>
+                                <usb:port-id>USB30-${id}</usb:port-id>
                                 <usb:version>USB3.0</usb:version>
                                 <usb:speed>5.00</usb:speed>

File: nuc_description/urdf/nuc.urdf.xacro (robot description, xacro)
@@ -4,6 +4,4 @@
     <xacro:include filename="$(find interface_description)/urdf/cat6.urdf.xacro"/>
     <xacro:include filename="$(find interface_description)/urdf/usb30.urdf.xacro"/>
-    <!-- <xacro:include filename="$(find interface_description)/urdf/wifi4.urdf.xacro"/> -->
-    <!-- <xacro:include filename="$(find interface_description)/urdf/wifi5.urdf.xacro"/> -->
     <xacro:macro name="nuc" params="parent id:=0 xyz:= '-1 1 0' ">
         <joint name="nuc_${id}_joint" type="fixed">
@@ -92,27 +90,25 @@
         <yang>
             <!-- NUC network topology -->
-            <!-- valahol ezen belül példányosítani kell az usb-t! -->
-            <!-- <xacro:usb30 parent="world" id="0"> -->
             <network>
-                <network-id>nuc-network</network-id>
+                <network-id>nuc-${id}-network</network-id>
                 <network-types>
                     <dl:device-layer-topology xmlns:dl="urn:ietf:params:xml:ns:yang:device-layer"/>
                 </network-types>
                 <supporting-network>
-                    <network-ref>nuc-supporting-network</network-ref>
+                    <network-ref>nuc-${id}-supporting-network</network-ref>
                 </supporting-network>
                 <node>
-                    <node-id>nuc-usb-node</node-id>
+                    <node-id>nuc-${id}-usb-node</node-id>
                     <supporting-node>
-                        <network-ref>nuc-usb-supporting-network</network-ref>
-                        <node-ref>nuc-usb-supporting-node</node-ref>
+                        <network-ref>nuc-${id}-usb-supporting-network</network-ref>
+                        <node-ref>nuc-${id}-usb-supporting-node</node-ref>
                     </supporting-node>
                     <xacro:usb30 parent="world" id="0" />
                 </node>
                 <node>
-                    <node-id>nuc-cat6-node</node-id>
+                    <node-id>nuc-${id}-cat6-node</node-id>
                     <supporting-node>
-                        <network-ref>nuc-cat6-supporting-network</network-ref>
-                        <node-ref>nuc-cat6-supporting-node</node-ref>
+                        <network-ref>nuc-${id}-cat6-supporting-network</network-ref>
+                        <node-ref>nuc-${id}-cat6-supporting-node</node-ref>
                     </supporting-node>
                     <xacro:cat6 parent="world" id="0" />
