Commit message: all dl node in 1 nw

File: example_config/urdf/system_config.urdf.xacro (robot description, xacro)
@@ -23,19 +23,25 @@
                 xmlns:dl="urn:ietf:params:xml:ns:yang:device-layer"/>
         </network-types>
-        <ietf-network-topology:link xmlns:ietf-network-topology="urn:ietf:params:xml:ns:yang:ietf-network-topology">
-            <ietf-network-topology:link-id>link-1</ietf-network-topology:link-id>
-            <ietf-network-topology:source>
-                <ietf-network-topology:source-node>node-1</ietf-network-topology:source-node>
-                <ietf-network-topology:source-tp>tp-1</ietf-network-topology:source-tp>
-            </ietf-network-topology:source>
-            <ietf-network-topology:destination>
-                <ietf-network-topology:dest-node>node-2</ietf-network-topology:dest-node>
-                <ietf-network-topology:dest-tp>tp-2</ietf-network-topology:dest-tp>
-            </ietf-network-topology:destination>
-            <device-layer:device-layer-link-attributes xmlns:device-layer="urn:ietf:params:xml:ns:yang:device-layer">
-                <device-layer:physical-link-name>Link-1</device-layer:physical-link-name>
-                <device-layer:physical-link-type>cat5e</device-layer:physical-link-type>
-            </device-layer:device-layer-link-attributes>
-        </ietf-network-topology:link>
+        <!-- instantiate d455 camera -->
+        <xacro:sensor_d455 parent="world">
+            <origin xyz="-0.022 -0.039 -0.01" rpy="0 1.57 0" />
+        </xacro:sensor_d455>
+        <!-- instantiate nuc -->
+        <xacro:nuc parent="world" id="0" />
+        <nt:link xmlns:nt="urn:ietf:params:xml:ns:yang:ietf-network-topology">
+            <nt:link-id>link-1</nt:link-id>
+            <nt:source>
+                <nt:source-node>node-1</nt:source-node>
+                <nt:source-tp>tp-1</nt:source-tp>
+            </nt:source>
+            <nt:destination>
+                <nt:dest-node>node-2</nt:dest-node>
+                <nt:dest-tp>tp-2</nt:dest-tp>
+            </nt:destination>
+            <dl:device-layer-link-attributes xmlns:dl="urn:ietf:params:xml:ns:yang:device-layer">
+                <dl:physical-link-name>Link-1</dl:physical-link-name>
+                <dl:physical-link-type>cat5e</dl:physical-link-type>
+            </dl:device-layer-link-attributes>
+        </nt:link>
     </network>
 </robot>

File: interface_description/urdf/cat6.urdf.xacro (robot description, xacro)
@@ -1,7 +1,4 @@
 <?xml version="1.0" encoding="UTF-8" ?>
 <robot xmlns:xacro="http://ros.org/wiki/xacro"
-       xmlns:ietf-network-topology="urn:ietf:params:xml:ns:yang:ietf-network-topology"
-       xmlns:device-layer="urn:ietf:params:xml:ns:yang:device-layer"
-       xmlns:ethernet-port="urn:ietf:params:xml:ns:yang:ethernet-port"
        name="cat6">
     <xacro:macro name="cat6" params="parent id:=0">
@@ -28,17 +25,17 @@
             </collision>
         </link>
-            <ietf-network-topology:termination-point xmlns:ietf-network-topology="urn:ietf:params:xml:ns:yang:ietf-network-topology">
-                <ietf-network-topology:tp-id>tp-1</ietf-network-topology:tp-id>
-                <device-layer:device-layer-termination-point-attributes xmlns:device-layer="urn:ietf:params:xml:ns:yang:device-layer">
-                    <device-layer:port-name>rj45-${id}</device-layer:port-name>
-                    <device-layer:port-type>rj45</device-layer:port-type>
-                    <ethernet-port:ethernet-port xmlns:ethernet-port="urn:ietf:params:xml:ns:yang:ethernet-port">
-                        <ethernet-port:port-id>eth-${id}</ethernet-port:port-id>
-                        <ethernet-port:mac-address>00:1A:2B:3C:4D:5E</ethernet-port:mac-address>
-                        <ethernet-port:speed>1Gbps</ethernet-port:speed>
-                        <ethernet-port:duplex-mode>full</ethernet-port:duplex-mode>
-                    </ethernet-port:ethernet-port>
-                </device-layer:device-layer-termination-point-attributes>
-            </ietf-network-topology:termination-point>
+        <nt:termination-point xmlns:nt="urn:ietf:params:xml:ns:yang:ietf-network-topology">
+            <nt:tp-id>tp-1</nt:tp-id>
+            <dl:device-layer-termination-point-attributes xmlns:dl="urn:ietf:params:xml:ns:yang:device-layer">
+                <dl:port-name>rj45-${id}</dl:port-name>
+                <dl:port-type>rj45</dl:port-type>
+                <eth:ethernet-port xmlns:eth="urn:ietf:params:xml:ns:yang:ethernet-port">
+                    <eth:port-id>eth-${id}</eth:port-id>
+                    <eth:mac-address>00:1A:2B:3C:4D:5E</eth:mac-address>
+                    <eth:speed>1Gbps</eth:speed>
+                    <eth:duplex-mode>full</eth:duplex-mode>
+                </eth:ethernet-port>
+            </dl:device-layer-termination-point-attributes>
+        </nt:termination-point>
     </xacro:macro>
 </robot>

File: interface_description/urdf/usb-typec.urdf.xacro (robot description, xacro)
@@ -1,7 +1,4 @@
 <?xml version="1.0" encoding="UTF-8" ?>
 <robot xmlns:xacro="http://ros.org/wiki/xacro"
-       xmlns:ietf-network-topology="urn:ietf:params:xml:ns:yang:ietf-network-topology"
-       xmlns:device-layer="urn:ietf:params:xml:ns:yang:device-layer"
-       xmlns:usb-port="urn:ietf:params:xml:ns:yang:usb-port"
        name="usb_typec">
     <xacro:macro name="usb_typec" params="parent id=0">
@@ -28,17 +25,17 @@
             </collision>
         </link>
-            <ietf-network-topology:termination-point xmlns:ietf-network-topology="urn:ietf:params:xml:ns:yang:ietf-network-topology">
-                <ietf-network-topology:tp-id>tp-1</ietf-network-topology:tp-id>
-                <device-layer:device-layer-termination-point-attributes xmlns:device-layer="urn:ietf:params:xml:ns:yang:device-layer">
-                    <device-layer:port-name>port-1</device-layer:port-name>
-                    <device-layer:port-type>usb-c</device-layer:port-type>
-                    <usb-port:usb-port xmlns:usb-port="urn:ietf:params:xml:ns:yang:usb-port">
-                        <usb-port:port-id>usb-typec-${id}</usb-port:port-id>
-                        <usb-port:version>USB3.2</usb-port:version>
-                        <usb-port:speed>5.00</usb-port:speed>
-                        <usb-port:power-consumption>2.5</usb-port:power-consumption>
-                    </usb-port:usb-port>
-                </device-layer:device-layer-termination-point-attributes>
-            </ietf-network-topology:termination-point>
+        <nt:termination-point xmlns:nt="urn:ietf:params:xml:ns:yang:ietf-network-topology">
+            <nt:tp-id>tp-1</nt:tp-id>
+            <dl:device-layer-termination-point-attributes xmlns:dl="urn:ietf:params:xml:ns:yang:device-layer">
+                <dl:port-name>port-1</dl:port-name>
+                <dl:port-type>usb-c</dl:port-type>
+                <usb:usb-port xmlns:usb="urn:ietf:params:xml:ns:yang:usb-port">
+                    <usb:port-id>usb-typec-${id}</usb:port-id>
+                    <usb:version>USB3.2</usb:version>
+                    <usb:speed>5.00</usb:speed>
+                    <usb:power-consumption>2.5</usb:power-consumption>
+                </usb:usb-port>
+            </dl:device-layer-termination-point-attributes>
+        </nt:termination-point>
     </xacro:macro>
 </robot>

File: interface_description/urdf/usb30.urdf.xacro (robot description, xacro)
@@ -1,7 +1,4 @@
 <?xml version="1.0" encoding="UTF-8" ?>
 <robot xmlns:xacro="http://ros.org/wiki/xacro"
-       xmlns:ietf-network-topology="urn:ietf:params:xml:ns:yang:ietf-network-topology"
-       xmlns:device-layer="urn:ietf:params:xml:ns:yang:device-layer"
-       xmlns:usb-port="urn:ietf:params:xml:ns:yang:usb-port"
        name="usb30">
     <xacro:macro name="usb30" params="parent id:=0">
@@ -28,17 +25,17 @@
             </collision>
         </link>
-            <ietf-network-topology:termination-point xmlns:ietf-network-topology="urn:ietf:params:xml:ns:yang:ietf-network-topology">
-                <ietf-network-topology:tp-id>tp-1</ietf-network-topology:tp-id>
-                <dl:device-layer-termination-point-attributes xmlns:dl="urn:ietf:params:xml:ns:yang:device-layer">
-                    <dl:port-name>port-1</dl:port-name>
-                    <dl:port-type>usb-a</dl:port-type>
-                    <usb:usb-port xmlns:usb="urn:ietf:params:xml:ns:yang:usb-port">
-                        <usb:port-id>USB30-${id}</usb:port-id>
-                        <usb:version>USB3.0</usb:version>
-                        <usb:speed>5.00</usb:speed>
-                        <usb:power-consumption>2.5</usb:power-consumption>
-                    </usb:usb-port>
-                </dl:device-layer-termination-point-attributes>
-            </ietf-network-topology:termination-point>
+        <nt:termination-point xmlns:nt="urn:ietf:params:xml:ns:yang:ietf-network-topology">
+            <nt:tp-id>tp-1</nt:tp-id>
+            <dl:device-layer-termination-point-attributes xmlns:dl="urn:ietf:params:xml:ns:yang:device-layer">
+                <dl:port-name>port-1</dl:port-name>
+                <dl:port-type>usb-a</dl:port-type>
+                <usb:usb-port xmlns:usb="urn:ietf:params:xml:ns:yang:usb-port">
+                    <usb:port-id>USB30-${id}</usb:port-id>
+                    <usb:version>USB3.0</usb:version>
+                    <usb:speed>5.00</usb:speed>
+                    <usb:power-consumption>2.5</usb:power-consumption>
+                </usb:usb-port>
+            </dl:device-layer-termination-point-attributes>
+        </nt:termination-point>
     </xacro:macro>
 </robot>

File: nuc_description/urdf/nuc.urdf.xacro (robot description, xacro)
@@ -4,5 +4,5 @@
     <xacro:include filename="$(find interface_description)/urdf/cat6.urdf.xacro"/>
     <xacro:include filename="$(find interface_description)/urdf/usb30.urdf.xacro"/>
-    <xacro:macro name="nuc" params="parent id:=0 xyz:= '-1 1 0' ">
+    <xacro:macro name="nuc" params="parent id:=0 xyz:='-1 1 0' ">
         <joint name="nuc_${id}_joint" type="fixed">
             <origin xyz="${xyz}" rpy="0 0 0" />
@@ -88,23 +88,17 @@
             </collision>
         </link>
-            <!-- NUC network topology -->
-            <network>
-                <network-id>nuc-${id}-network</network-id>
-                <network-types>
-                    <dl:device-layer-topology xmlns:dl="urn:ietf:params:xml:ns:yang:device-layer"/>
-                </network-types>
-                <node>
-                    <node-id>nuc-${id}-usb-node</node-id>
-                    <xacro:usb30 parent="world" id="0" />
-                </node>
-                <node>
-                    <node-id>nuc-${id}-cat6-node</node-id>
-                    <dl:device-layer-node-attributes xmlns:dl="urn:ietf:params:xml:ns:yang:device-layer">
-                        <dl:device-name>nuc-${id}</dl:device-name>
-                        <dl:device-type>pc</dl:device-type>
-                    </dl:device-layer-node-attributes>
-                    <xacro:cat6 parent="world" id="0" />
-                </node>
-            </network>
+        <!-- NUC network topology -->
+        <node>
+            <node-id>nuc-${id}-usb-node</node-id>
+            <xacro:usb30 parent="world" id="0" />
+        </node>
+        <node>
+            <node-id>nuc-${id}-cat6-node</node-id>
+            <dl:device-layer-node-attributes xmlns:dl="urn:ietf:params:xml:ns:yang:device-layer">
+                <dl:device-name>nuc-${id}</dl:device-name>
+                <dl:device-type>pc</dl:device-type>
+            </dl:device-layer-node-attributes>
+            <xacro:cat6 parent="world" id="0" />
+        </node>
     </xacro:macro>
 </robot>

Commit message: yang content update

File: example_config/urdf/system_config.urdf.xacro (robot description, xacro)
@@ -11,10 +11,4 @@
     <!-- import d455 camera -->
     <xacro:include filename="$(find realsense2_description)/urdf/_d455.urdf.xacro" />
-    <!-- instantiate d455 camera -->
-    <xacro:sensor_d455 parent="world">
-        <origin xyz="-0.022 -0.039 -0.01" rpy="0 1.57 0" />
-    </xacro:sensor_d455>
-    <!-- instantiate nuc -->
-    <xacro:nuc parent="world" id="0" />
     <network>
         <network-id>device-layer-network</network-id>
@@ -24,9 +18,9 @@
         </network-types>
         <!-- instantiate d455 camera -->
-        <xacro:sensor_d455 parent="world">
+        <xacro:sensor_d455 parent="world" id="0">
             <origin xyz="-0.022 -0.039 -0.01" rpy="0 1.57 0" />
         </xacro:sensor_d455>
         <!-- instantiate nuc -->
-        <xacro:nuc parent="world" id="0" />
+        <xacro:nuc parent="world" id="0" origin_xyz="-1 1 0"/>
         <nt:link xmlns:nt="urn:ietf:params:xml:ns:yang:ietf-network-topology">
             <nt:link-id>link-1</nt:link-id>

Commit message: ur & controlbox added

File: example_config/urdf/system_config.urdf.xacro (robot description, xacro)
@@ -12,6 +12,10 @@
     <!-- import d455 camera -->
     <xacro:include filename="$(find realsense2_description)/urdf/_d455.urdf.xacro" />
+    <!-- import usb-cable -->
+    <xacro:include filename="$(find cable_description)/urdf/usb-cable.urdf.xacro" />
     <!-- import ethernet-cable -->
-    <xacro:include filename="$(find cable_description)/urdf/usb-cable.urdf.xacro" />
+    <xacro:include filename="$(find cable_description)/urdf/ethernet-cable.urdf.xacro" />
+    <!-- import universal robots ur3e -->
+    <xacro:include filename="$(find ur_description)/urdf/ur_macro.xacro" />
     <!-- Device definition in a network -->
     <network>
@@ -22,4 +26,15 @@
         <!-- instantiate nuc -->
         <xacro:nuc parent="world" id="0" origin_xyz="-1 1 0"/>
+        <!-- instantiate universal robots ur3e -->
+        <xacro:ur_robot
+            name="ur3e"
+            tf_prefix=""
+            parent="world"
+            joint_limits_parameters_file="$(find ur_description)/config/ur3e/joint_limits.yaml"
+            kinematics_parameters_file="$(find ur_description)/config/ur3e/default_kinematics.yaml"
+            physical_parameters_file="$(find ur_description)/config/ur3e/physical_parameters.yaml"
+            visual_parameters_file="$(find ur_description)/config/ur3e/visual_parameters.yaml">
+            <origin xyz="0 0 0" rpy="0 0 0" />
+        </xacro:ur_robot>
         <!-- instantiate d455 camera -->
         <xacro:sensor_d455 parent="world" id="0">
@@ -27,5 +42,6 @@
         </xacro:sensor_d455>
         <!-- instantiate ethernet-cable -->
-        <xacro:usb-cable parent="nuc-0-cat6-0-link" src_node="nuc-0" dst_node="d455" src_tp="cat6-0" dst_tp="usb-typec-0" link_type="usb30" length="2"/>
+        <!-- <xacro:ethernet-cable parent="nuc-0-usb30-0-link" src_node="nuc-0" dst_node="d455" src_tp="usb30-0" dst_tp="usb-typec-0" link_type="usb30" length="2"/> -->
+        <xacro:usb-cable parent="nuc-0-usb30-0-link" src_node="nuc-0" dst_node="d455" src_tp="usb30-0" dst_tp="usb-typec-0" link_type="usb30" length="2"/>
     </network>
     <network xmlns:nw="urn:ietf:params:xml:ns:yang:ietf-network">
@@ -37,6 +53,6 @@
             <nw:network-ref>device-layer-network</nw:network-ref>
         </nw:supporting-network>
-        <nw:node>
-            <nw:node-id>nuc-supporting</nw:node-id>
+        <node>
+            <node-id>nuc-supporting</node-id>
             <nw:supporting-node>
                 <nw:network-ref>device-layer-network</nw:network-ref>
@@ -61,5 +77,5 @@
                 </nl:network-layer-termination-point-attributes>
             </nt:termination-point>
-        </nw:node>
+        </node>
     </network>
 </robot>

Commit message: namespaces fixed

File: example_config/urdf/system_config.urdf.xacro (robot description, xacro)
@@ -2,9 +2,5 @@
 <robot name="example-configuration"
       xmlns:xacro="http://wiki.ros.org/xacro"
-      xmlns:dl="urn:ietf:params:xml:ns:yang:device-layer"
-      xmlns:nl="urn:ietf:params:xml:ns:yang:network-layer"
-      xmlns:nt="urn:ietf:params:xml:ns:yang:ietf-network-topology"
-      xmlns:nw="urn:ietf:params:xml:ns:yang:ietf-network"
-      xmlns:usb="urn:ietf:params:xml:ns:yang:usb-port">
+      >
     <link name="world" />
     <!-- import nuc -->
@@ -39,5 +35,5 @@
         <!-- instantiate d455 camera -->
         <xacro:sensor_d455 parent="world" id="0">
-            <origin xyz="-0.022 -0.039 -0.01" rpy="0 1.57 0" />
+            <origin xyz="1 -1 0" rpy="0 1.57 0" />
         </xacro:sensor_d455>
         <!-- instantiate ethernet-cable -->
